Commit message: some fixes

File: cob_3d_mapping_demonstrator/md.urdf.xacro (robot description, xacro)
@@ -1,4 +1,5 @@
 <?xml version="1.0"?>
 <robot name="mapping_demonstrator">
+	<link name="map"/>
 	<!-- BASE LINK is the lower case-->
 	<link name="base"/>
@@ -72,5 +73,5 @@
 		-->
 		<link name="tilt"/>
-		<link name="camera"/>
+		<link name="camera_link"/>
 			<!--inertial>
 				<origin xyz="0 0 0" rpy="0 0 0"/>
@@ -116,8 +117,13 @@
 			</collision-->
 		<!--/link-->
+		<joint name="map_base" type="fixed">
+			<parent link="map"/>
+			<child link="base" />
+			<origin xyz="0 0 0" rpy="0 0 0"/>
+		</joint>
 		<joint name="stepper" type="revolute">
 			<parent link="base"/>
 			<child link="pan" />
-			<origin xyz="0 0 0.06" rpy="0 3.14 0"/>
+			<origin xyz="0 0 1.42" rpy="0 3.14 0"/>
 			<limit lower="-7" upper="7" velocity="1.02" effort="0"/>
 			<!--calibration rising="-0.9"/-->
@@ -129,16 +135,16 @@
 			<parent link="pan"/>
 			<child link="tilt"/>
-			<origin xyz="0 0 0.066" rpy="1.57 0 0"/>
-			<axis xyz="0 1 0"/>
+			<origin xyz="0 0 -0.066" rpy="-1.57 0 0"/>
+			<axis xyz="0 0 1"/>
 			<limit lower="-1.56" upper="1.56" velocity="1.02" effort="0"/>
 			<!-- max vel is 12.31-->
-			<!--calibration rising="0.04"/-->
-			<calibration rising="0"/>
+			<calibration rising="0.04"/>
+			<!--calibration rising="0"/-->
 			<!--max vel is 12.32 -->
-		</joint >
+		</joint>
 		<joint name="camjoint" type="fixed">
 			<parent link="tilt"/>
-			<child link="camera"/>
-			<origin xyz="0 0 0" rpy="0 0 0"/>
+			<child link="camera_link"/>
+			<origin xyz="0 0.07 0" rpy="-1.57 0 0"/>
 		</joint>
 </robot>

Commit message: changed urdf

File: cob_3d_mapping_demonstrator/md.urdf.xacro (robot description, xacro)
@@ -1,4 +1,6 @@
 <?xml version="1.0"?>
-<robot name="mapping_demonstrator">
+<robot name="mapping_demonstrator" xmlns:xacro="http://ros.org/wiki/xacro">
+<property name="M_PI" value="3.14159"/>
+<xacro:macro name="map_demo">
 	<link name="map"/>
 	<!-- BASE LINK is the lower case-->
@@ -73,5 +75,5 @@
 		-->
 		<link name="tilt"/>
-		<link name="camera_link"/>
+		<!--link name="camera_link"/-->
 			<!--inertial>
 				<origin xyz="0 0 0" rpy="0 0 0"/>
@@ -146,5 +148,90 @@
 			<parent link="tilt"/>
 			<child link="camera_link"/>
-			<origin xyz="0 0.07 0" rpy="-1.57 0 0"/>
-		</joint>
+			<origin xyz="0 0.068 -0.0075" rpy="-1.57 0 0"/>
+		</joint>
+		  <!--joint name="base_camera_joint" type="fixed">
+    <origin xyz="${turtlebot_calib_cam_x} ${turtlebot_calib_cam_y} 0.124"
+            rpy="${turtlebot_calib_cam_rr} ${turtlebot_calib_cam_rp} ${turtlebot_calib_cam_ry}" />
+    <parent link="${turtlebot_camera_parent_name}" />
+    <child link="camera_link" />
+  </joint-->
+  <link name="camera_link">
+    <inertial>
+      <mass value="0.01" />
+      <origin xyz="0 0 0" />
+      <inertia ixx="0.001" ixy="0.0" ixz="0.0"
+        iyy="0.001" iyz="0.0"
+        izz="0.001" />
+    </inertial>
+    <visual>
+      <origin xyz=" 0 0 0 " rpy="0 0 0" />
+      <geometry>
+        <mesh filename="package://turtlebot_description/meshes/kinect.dae"/>
+      </geometry>
+    </visual>
+    <collision>
+      <origin xyz="0.0 0.0 0.0" rpy="0 0 0" />
+      <geometry>
+        <box size="0.0730 .2760 0.0720"/>
+      </geometry>
+    </collision>
+  </link>
+  <joint name="camera_depth_joint" type="fixed">
+    <origin xyz="0 0.049 0" rpy="0 0 0" />
+    <parent link="camera_link" />
+    <child link="camera_depth_frame" />
+  </joint>
+  <link name="camera_depth_frame">
+    <inertial>
+      <mass value="0.01" />
+      <origin xyz="0 0 0" />
+      <inertia ixx="0.001" ixy="0.0" ixz="0.0"
+        iyy="0.001" iyz="0.0"
+        izz="0.001" />
+    </inertial>
+  </link>
+  <joint name="camera_depth_optical_joint" type="fixed">
+    <origin xyz="0 0 0" rpy="${-M_PI/2} 0 ${-M_PI/2}" />
+    <parent link="camera_depth_frame" />
+    <child link="camera_depth_optical_frame" />
+  </joint>
+  <link name="camera_depth_optical_frame">
+    <inertial>
+      <mass value="0.001" />
+      <origin xyz="0 0 0" />
+      <inertia ixx="0.0001" ixy="0.0" ixz="0.0"
+        iyy="0.0001" iyz="0.0"
+        izz="0.0001" />
+    </inertial>
+  </link>
+  <joint name="camera_rgb_joint" type="fixed">
+    <origin xyz="0 0.022 0" rpy="0 0 0" />
+    <parent link="camera_link" />
+    <child link="camera_rgb_frame" />
+  </joint>
+  <link name="camera_rgb_frame">
+    <inertial>
+      <mass value="0.001" />
+      <origin xyz="0 0 0" />
+      <inertia ixx="0.0001" ixy="0.0" ixz="0.0"
+        iyy="0.0001" iyz="0.0"
+        izz="0.0001" />
+    </inertial>
+  </link>
+  <joint name="camera_rgb_optical_joint" type="fixed">
+    <origin xyz="0 0 0" rpy="${-M_PI/2} 0 ${-M_PI/2}" />
+    <parent link="camera_rgb_frame" />
+    <child link="camera_rgb_optical_frame" />
+  </joint>
+  <link name="camera_rgb_optical_frame">
+    <inertial>
+      <mass value="0.001" />
+      <origin xyz="0 0 0" />
+      <inertia ixx="0.0001" ixy="0.0" ixz="0.0"
+        iyy="0.0001" iyz="0.0"
+        izz="0.0001" />
+    </inertial>
+  </link>
+</xacro:macro>
+<xacro:map_demo/>
 </robot>
